File: LCDButtonBooster/spi_lcd_booster_dip_v3.brd (EAGLE design)
At the start: 49.6 x 49.7 mm, 28 parts, among them IC1 REG1117

Commit message: Various changes
Other:
- board text added: "1/7/2012"
- board text added: "v3"
- board text removed: "1/5/2012"
- board text removed: "D50554_2_20boards"
- board text removed: "v2"
Changed lines of the file:
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@@
 <wire x1="50.17" y1="50.09" x2="0.6" y2="50.09" width="0" layer="20"/>
 <wire x1="0.6" y1="50.09" x2="0.6" y2="0.4" width="0" layer="20"/>
-<text x="6.985" y="22.86" size="1.4224" layer="21" rot="R90">1/5/2012</text>
+<text x="6.985" y="22.86" size="1.4224" layer="21" rot="R90">1/7/2012</text>
 <text x="39.37" y="23.1775" size="1.4224" layer="22" rot="MR0">LCD-Button-Boosterpack</text>
 <text x="39.37" y="41.91" size="1.778" layer="22" rot="MR0">apus.pro</text>
@@
 <wire x1="46.99" y1="41.91" x2="49.53" y2="41.91" width="0.254" layer="21"/>
 <wire x1="49.53" y1="41.91" x2="49.53" y2="49.53" width="0.254" layer="21"/>
-<text x="6.985" y="17.78" size="1.4224" layer="21" rot="R90">v2</text>
-<text x="39.37" y="20.32" size="1.778" layer="22" rot="MR0">v2</text>
+<text x="39.37" y="20.32" size="1.778" layer="22" rot="MR0">v3</text>
 <text x="44.45" y="12.7" size="1.778" layer="22" rot="MR0">http://lars.roland.bz/lcd/</text>
-<text x="45.72" y="2.54" size="1.778" layer="21">v2</text>
+<text x="45.72" y="2.54" size="1.778" layer="21">v3</text>
 <text x="45.4025" y="44.7675" size="1.778" layer="21">+</text>
 <text x="45.4025" y="42.2275" size="1.778" layer="21">-</text>
 <text x="45.4025" y="47.625" size="1.778" layer="21">-</text>
-<text x="12.3825" y="43.18" size="1.778" layer="21">D50554_2_20boards</text>
 </plain>
 <attributes>
@@
 <contactref element="C2" pad="1"/>
 <contactref element="U$1" pad="10"/>
-<wire x1="22.4825" y1="29.6875" x2="22.4825" y2="33.3975" width="0.254" layer="1"/>
-<wire x1="22.4825" y1="33.3975" x2="21.59" y2="34.29" width="0.254" layer="1"/>
+<wire x1="22.4825" y1="29.6875" x2="22.4825" y2="32.1275" width="0.254" layer="1"/>
+<wire x1="22.4825" y1="32.1275" x2="21.59" y2="34.29" width="0.254" layer="1"/>
 <via x="21.59" y="34.29" extent="1-16" drill="0.3048" shape="square"/>
 <wire x1="21.59" y1="34.29" x2="21.59" y2="36.83" width="0.254" layer="16"/>
@@
 <contactref element="C2" pad="2"/>
 <contactref element="U$1" pad="9"/>
-<wire x1="23.2825" y1="29.6875" x2="23.2825" y2="33.8675" width="0.254" layer="1"/>
-<wire x1="23.2825" y1="33.8675" x2="22.86" y2="34.29" width="0.254" layer="1"/>
+<wire x1="23.2825" y1="29.6875" x2="23.2825" y2="32.5975" width="0.254" layer="1"/>
+<wire x1="23.2825" y1="32.5975" x2="22.86" y2="34.29" width="0.254" layer="1"/>
 <via x="22.86" y="34.29" extent="1-16" drill="0.3048" shape="square"/>
 <wire x1="21.16" y1="39.81" x2="22.86" y2="38.1" width="0.254" layer="16"/>
@@
 <wire x1="40.64" y1="26.518" x2="41.758" y2="25.4" width="0.254" layer="16"/>
 <contactref element="U$1" pad="11"/>
-<wire x1="21.6825" y1="29.6875" x2="21.6825" y2="32.9275" width="0.254" layer="1"/>
-<wire x1="21.6825" y1="32.9275" x2="19.05" y2="35.56" width="0.254" layer="1"/>
+<wire x1="21.6825" y1="29.6875" x2="21.6825" y2="31.6575" width="0.254" layer="1"/>
+<wire x1="21.6825" y1="31.6575" x2="19.05" y2="35.56" width="0.254" layer="1"/>
 <via x="19.05" y="35.56" extent="1-16" drill="0.3048" shape="square"/>
 <wire x1="19.05" y1="35.56" x2="12.7" y2="35.56" width="0.254" layer="1"/>
@@
 <via x="13.97" y="41.91" extent="1-16" drill="0.3048" shape="square"/>
 <wire x1="13.97" y1="41.91" x2="26.67" y2="41.91" width="0.254" layer="1"/>
-<wire x1="24.8825" y1="29.6875" x2="24.8825" y2="33.7725" width="0.254" layer="1"/>
-<wire x1="24.8825" y1="33.7725" x2="25.4" y2="34.29" width="0.254" layer="1"/>
+<wire x1="24.8825" y1="29.6875" x2="24.8825" y2="32.5025" width="0.254" layer="1"/>
+<wire x1="24.8825" y1="32.5025" x2="25.4" y2="34.29" width="0.254" layer="1"/>
 <via x="25.4" y="34.29" extent="1-16" drill="0.3048" shape="square"/>
 <via x="26.67" y="41.91" extent="1-16" drill="0.3048" shape="square"/>
