File: LCDButtonBooster/spi_lcd_booster_dip_v3.sch (EAGLE design)
At the start: 28 parts, among them IC1 REG1117

Commit message: Various changes
Changed lines of the file:
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@@
 <pinref part="IC1" gate="G$1" pin="VOUT"/>
 <junction x="22.86" y="5.08"/>
+<junction x="7.62" y="25.4"/>
+<junction x="104.14" y="71.12"/>
 </segment>
 </net>
@@
 <wire x1="203.2" y1="15.24" x2="203.2" y2="33.02" width="0.1524" layer="91"/>
 <junction x="40.64" y="20.32"/>
+<junction x="7.62" y="20.32"/>
 </segment>
 </net>
@@
 <pinref part="LEDSW" gate="G$1" pin="1"/>
 <wire x1="165.1" y1="35.56" x2="187.96" y2="35.56" width="0.1524" layer="91"/>
+<junction x="165.1" y="35.56"/>
 </segment>
 </net>
@@
 <pinref part="IC1" gate="G$1" pin="VIN"/>
 <junction x="-2.54" y="5.08"/>
-</segment>
-</net>
+<junction x="0" y="-15.24"/>
+</segment>
+</net>
